File: stm32f4_uno_poe.kicad_pcb (KiCad board)
At the start: 2 copper layers, 68.6 x 53.3 mm, 55 parts, among them J104 STM32 GPIO, J106 Power, J107 Conn_01x04, J108 Ethernet, J111 Analog, J112 Barrel_Jack, U201 TCMT1107, U202 CJ431, U203 TPS23754PWP

Commit message: WIP
Parts:
- added C214: 2u2 100V, Capacitor_SMD:C_1206_3216Metric, F.Cu at (203.8, 92.2)
- added C215: 100n 100V, Capacitor_SMD:C_0805_2012Metric, F.Cu at (187.8, 87.8)
- added C216: 100p 500V, Capacitor_SMD:C_0805_2012Metric, F.Cu at (187.8, 90.8)
- added C225: 100n 100V, Capacitor_SMD:C_0805_2012Metric, F.Cu at (187.8, 93.8)
- added C227: 22u 25V, Capacitor_SMD:C_0805_2012Metric, F.Cu at (187.8, 96.9)
- added C228: 1u 50V, Capacitor_SMD:C_0805_2012Metric, F.Cu at (187.8, 99.9)
- added C229: 100n 100V, Capacitor_SMD:C_0805_2012Metric, F.Cu at (187.8, 102.9)
- added D206: 1N4148WS, Diode_SMD:D_SOD-323, F.Cu at (187.8, 105.9)
- added D214: 64V TVS, Diode_SMD:D_SMC, F.Cu at (195.5, 90.2)
- added L205: 3u3, Inductor_SMD:L_Sunlord_SWPA4030S, F.Cu at (205.1, 101.8)
- added Q201: Si7450DP, Package_SO:PowerPAK_SO-8_Single, F.Cu at (198.2, 102.2)
- added R221: 39k, Resistor_SMD:R_0805_2012Metric, F.Cu at (205.0, 95.5)
- added R222: 100, Resistor_SMD:R_0603_1608Metric, F.Cu at (192.1, 95.3)
- added R223: 4E7, Resistor_SMD:R_0603_1608Metric, F.Cu at (192.1, 97.8)
- added R224: 1k, Resistor_SMD:R_0603_1608Metric, F.Cu at (192.1, 100.3)
- added R225: 274k, Resistor_SMD:R_0603_1608Metric, F.Cu at (192.1, 102.9)
- added R226: 0E12 1W, Resistor_SMD:R_2512_6332Metric, F.Cu at (198.4, 96.5)
- added R227: 75 750mW, Resistor_SMD:R_2010_5025Metric, F.Cu at (204.7, 88.4)
- C207, C213: value 100n 100V -> 2u2 100V; footprint Capacitor_SMD:C_0805_2012Metric -> Capacitor_SMD:C_1206_3216Metric
- C211: value 1u 50V -> 47u 63V; footprint Capacitor_SMD:C_0805_2012Metric -> Capacitor_SMD:C_Elec_8x10.2
- D205: value 64V TVS -> 1A 200V 35ns; footprint Diode_SMD:D_SMC -> Diode_SMD:D_SMA
Connections:
- C207 pad 1: /PoE/PGND -> /PoE/VDD
- C207 pad 2: /PoE/VB -> /PoE/PGND
- C211 pad 1: Net-(U203-VC) -> /PoE/VDD
- C213 pad 1: /PoE/VDD -> Net-(C213-Pad1)
- C213 pad 2: /PoE/VSS -> /PoE/PGND
- D205 pad 1: /PoE/VDD -> Net-(D205-K)
- D205 pad 2: /PoE/VSS -> Net-(D205-A)
- U203 pad 3: unconnected-(U203-CS-Pad3) -> /PoE/CS
- U203 pad 5: unconnected-(U203-GATE-Pad5) -> /PoE/GATE
- U203 pad 6: Net-(U203-VC) -> /PoE/VC

Commit message: Add flyback transformator
Parts:
- added TR201: Coilcraft POE40Q-xxE, Project_Library:Coilcraft POE40Q-xxE, F.Cu at (160.2, 79.7)
Changed lines of the file:
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@@
   (net 75 "/PoE/GATE")
   (net 76 "/PoE/CS")
+  (net 77 "unconnected-(TR201-Pad1)")
+  (net 78 "unconnected-(TR201-Pad2)")
+  (net 79 "unconnected-(TR201-Pad3)")
+  (net 80 "unconnected-(TR201-Pad4)")
+  (net 81 "unconnected-(TR201-Pad5)")
+  (net 82 "unconnected-(TR201-Pad6)")
+  (net 83 "unconnected-(TR201-Pad7)")
+  (net 84 "unconnected-(TR201-Pad8)")
+  (net 85 "unconnected-(TR201-Pad9)")
+  (net 86 "unconnected-(TR201-Pad10)")
   (footprint "Connector_PinSocket_2.54mm:PinSocket_1x08_P2.54mm_Vertical" locked (layer "F.Cu")
     (at 127.94 97.46 90)
@@
     )
   )
+  (footprint "Project_Library:Coilcraft POE40Q-xxE" (layer "F.Cu")
+    (at 160.1978 79.6798 90)
+    (property "Manufacturer" "Coilcraft")
+    (property "Sheetfile" "poe.kicad_sch")
+    (property "Sheetname" "PoE")
+    (property "ki_description" "Flyback Transformer, PCB")
+    (property "ki_keywords" "PCB Flyback Transformer")
+    (attr smd)
+    (fp_text reference "TR201" (at 0 -8.255 90) (layer "F.SilkS")
+        (effects (font (size 1 1) (thickness 0.15)))
+    )
+    (fp_text value "Coilcraft POE40Q-xxE" (at 0.254 6.595 90) (layer "F.Fab")
+        (effects (font (size 1 1) (thickness 0.15)))
+    )
+    (fp_line (start -9.53 -6.447) (end -8.73 -7.247)
+      (stroke (width 0.12) (type default)) (layer "F.SilkS"))
+    (fp_line (start -9.53 7.323) (end -9.53 -6.447)
+      (stroke (width 0.12) (type default)) (layer "F.SilkS"))
+    (fp_line (start -8.73 -7.247) (end 9.53 -7.247)
+      (stroke (width 0.12) (type default)) (layer "F.SilkS"))
+    (fp_line (start 9.53 -7.247) (end 9.53 7.323)
+      (stroke (width 0.12) (type default)) (layer "F.SilkS"))
+    (fp_line (start 9.53 7.323) (end -9.53 7.323)
+      (stroke (width 0.12) (type default)) (layer "F.SilkS"))
+    (fp_line (start -9.28 -5.842) (end 9.28 -5.842)
+      (stroke (width 0.05) (type default)) (layer "F.CrtYd"))
+    (fp_line (start -9.28 5.918) (end -9.28 -5.842)
+      (stroke (width 0.05) (type default)) (layer "F.CrtYd"))
+    (fp_line (start 9.28 -5.842) (end 9.28 5.918)
+      (stroke (width 0.05) (type default)) (layer "F.CrtYd"))
+    (fp_line (start 9.28 5.918) (end -9.28 5.918)
+      (stroke (width 0.05) (type default)) (layer "F.CrtYd"))
+    (pad "1" smd rect (at -8.255 -4.962) (size 1.27 1.55) (layers "F.Cu" "F.Paste" "F.Mask")
+      (net 77 "unconnected-(TR201-Pad1)") (pintype "passive") (thermal_bridge_angle 45))
+    (pad "2" smd rect (at -8.255 -2.462) (size 1.27 1.55) (layers "F.Cu" "F.Paste" "F.Mask")
+      (net 78 "unconnected-(TR201-Pad2)") (pintype "no_connect") (thermal_bridge_angle 45))
+    (pad "3" smd rect (at -8.255 0.038) (size 1.27 1.55) (layers "F.Cu" "F.Paste" "F.Mask")
+      (net 79 "unconnected-(TR201-Pad3)") (pintype "passive") (thermal_bridge_angle 45))
+    (pad "4" smd rect (at -8.255 2.538) (size 1.27 1.55) (layers "F.Cu" "F.Paste" "F.Mask")
+      (net 80 "unconnected-(TR201-Pad4)") (pintype "passive") (thermal_bridge_angle 45))
+    (pad "5" smd rect (at -8.255 5.038) (size 1.27 1.55) (layers "F.Cu" "F.Paste" "F.Mask")
+      (net 81 "unconnected-(TR201-Pad5)") (pintype "passive") (thermal_bridge_angle 45))
+    (pad "6" smd rect (at 8.255 5.038) (size 1.27 1.55) (layers "F.Cu" "F.Paste" "F.Mask")
+      (net 82 "unconnected-(TR201-Pad6)") (pintype "passive") (thermal_bridge_angle 45))
+    (pad "7" smd rect (at 8.255 2.538) (size 1.27 1.55) (layers "F.Cu" "F.Paste" "F.Mask")
+      (net 83 "unconnected-(TR201-Pad7)") (pintype "passive") (thermal_bridge_angle 45))
+    (pad "8" smd rect (at 8.255 0.038) (size 1.27 1.55) (layers "F.Cu" "F.Paste" "F.Mask")
+      (net 84 "unconnected-(TR201-Pad8)") (pintype "no_connect") (thermal_bridge_angle 45))
+    (pad "9" smd rect (at 8.255 -2.462) (size 1.27 1.55) (layers "F.Cu" "F.Paste" "F.Mask")
+      (net 85 "unconnected-(TR201-Pad9)") (pintype "passive") (thermal_bridge_angle 45))
+    (pad "10" smd rect (at 8.255 -4.962) (size 1.27 1.55) (layers "F.Cu" "F.Paste" "F.Mask")
+      (net 86 "unconnected-(TR201-Pad10)") (pintype "passive") (thermal_bridge_angle 45))
+    (model "${KIPRJMOD}/Project_Library.3dshapes/Coilcraft-POE40Q-XXX.step"
+      (offset (xyz 0 0 0))
+      (scale (xyz 1 1 1))
+      (rotate (xyz -90 0 0))
+    )
+  )

Commit message: WIP
Parts:
- added C217: 1n 2kV, Capacitor_SMD:C_1206_3216Metric, F.Cu at (221.8, 56.4)
- added C218: 1n 2kV, Capacitor_SMD:C_1206_3216Metric, F.Cu at (221.8, 59.7)
- added C219: 1u 50V, Capacitor_SMD:C_0603_1608Metric, F.Cu at (236.6, 55.9)
- added C220: 1n 2kV, Capacitor_SMD:C_1206_3216Metric, F.Cu at (221.8, 63.1)
- added C221: 1n 2kV, Capacitor_SMD:C_1206_3216Metric, F.Cu at (221.8, 66.4)
- added C222: 330p 500V, Capacitor_SMD:C_0805_2012Metric, F.Cu at (234.3, 78.3)
- added C223: 4u7 50V, Capacitor_SMD:C_1206_3216Metric, F.Cu at (221.8, 69.8)
- added C224: 4u7 50V, Capacitor_SMD:C_1206_3216Metric, F.Cu at (221.8, 73.1)
- added C226: 4u7 50V, Capacitor_SMD:C_1206_3216Metric, F.Cu at (221.8, 76.5)
- added C230: 4u7 50V, Capacitor_SMD:C_1206_3216Metric, F.Cu at (221.8, 79.8)
- added C231: 22u 63V, Capacitor_SMD:C_Elec_6.3x5.4, F.Cu at (229.6, 58.8)
- added C232: 1u 50V, Capacitor_SMD:C_0603_1608Metric, F.Cu at (236.6, 58.5)
- added D207: 1N4148WS, Diode_SMD:D_SOD-323, F.Cu at (235.3, 64.3)
- added D208: 150V 10A, Package_TO_SOT_SMD:TO-277A, F.Cu at (235.2, 72.7)
- added R228: 20, Resistor_SMD:R_0805_2012Metric, F.Cu at (226.8, 78.4)
- added R229: 100 750mW, Resistor_SMD:R_2010_5025Metric, F.Cu at (228.3, 70.6)
- added R230: 100 750mW, Resistor_SMD:R_2010_5025Metric, F.Cu at (228.3, 74.8)
- added R231: 10k, Resistor_SMD:R_0603_1608Metric, F.Cu at (236.6, 61.0)
- added U204: EL357N(C)(TA)-G, Package_SO:SOP-4_3.8x4.1mm_P2.54mm, F.Cu at (228.9, 65.7)
Connections:
- TR201 pad 1: unconnected-(TR201-Pad1) -> Net-(C213-Pad1)
- TR201 pad 10: unconnected-(TR201-Pad10) -> GND
- TR201 pad 3: unconnected-(TR201-Pad3) -> Net-(D205-A)
- TR201 pad 4: unconnected-(TR201-Pad4) -> /PoE/PGND
- TR201 pad 5: unconnected-(TR201-Pad5) -> Net-(R228-Pad1)
- TR201 pad 6: unconnected-(TR201-Pad6) -> Net-(D208-A-Pad1)
- TR201 pad 7: unconnected-(TR201-Pad7) -> Net-(D208-A-Pad1)
- TR201 pad 9: unconnected-(TR201-Pad9) -> GND

Commit message: Add ETH_RXER
Connections:
- J104 pad 1: /PB14 -> GND
- J108 pad 1: GND -> /ETH_RXER
Changed lines of the file:
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@@
   (net 21 "/PE12")
   (net 22 "/PE14")
-  (net 23 "/PB14")
+  (net 23 "/ETH_RXER")
   (net 24 "/PE3")
   (net 25 "/PE5")
@@
       (stroke (width 0.1) (type solid)) (layer "F.Fab"))
     (pad "1" thru_hole rect locked (at 0 0 90) (size 1.7 1.7) (drill 1) (layers "*.Cu" "*.Mask")
-      (net 1 "GND") (pinfunction "Pin_1") (pintype "passive"))
+      (net 23 "/ETH_RXER") (pinfunction "Pin_1") (pintype "passive+no_connect"))
     (pad "2" thru_hole oval locked (at 0 2.54 90) (size 1.7 1.7) (drill 1) (layers "*.Cu" "*.Mask")
       (net 15 "/ETH_TXD1") (pinfunction "Pin_2") (pintype "passive+no_connect"))
@@
       (stroke (width 0.1) (type solid)) (layer "F.Fab"))
     (pad "1" thru_hole rect locked (at 0 0 90) (size 1.7 1.7) (drill 1) (layers "*.Cu" "*.Mask")
-      (net 23 "/PB14") (pinfunction "Pin_1") (pintype "passive+no_connect"))
+      (net 1 "GND") (pinfunction "Pin_1") (pintype "passive"))
     (pad "2" thru_hole oval locked (at 0 2.54 90) (size 1.7 1.7) (drill 1) (layers "*.Cu" "*.Mask")
       (net 22 "/PE14") (pinfunction "Pin_2") (pintype "passive+no_connect"))

Commit message: #1 Use new central library KiCad-Lib
Parts:
- added J113: Conn_01x02, Connector_PinHeader_2.54mm:PinHeader_1x02_P2.54mm_Vertical, F.Cu at (221.4, 92.4)
- TR201: footprint Project_Library:Coilcraft POE40Q-xxE -> #Transformer:Coilcraft POE40Q-xxE
Connections:
- net /PoE/SHIELD renamed Earth
Changed lines of the file:
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@@
   (net 37 "/PoE/VB")
   (net 38 "/PoE/VDD")
-  (net 39 "/PoE/SHIELD")
+  (net 39 "Earth")
   (net 40 "/PoE/VDD_B")
   (net 41 "/PoE/VSS_B")
@@
       (stroke (width 0.1) (type solid)) (layer "F.Fab"))
     (pad "1" smd roundrect (at -1.475 0 180) (size 1.15 1.8) (layers "F.Cu" "F.Paste" "F.Mask") (roundrect_rratio 0.217391)
-      (net 39 "/PoE/SHIELD") (pintype "passive"))
+      (net 39 "Earth") (pintype "passive"))
     (pad "2" smd roundrect (at 1.475 0 180) (size 1.15 1.8) (layers "F.Cu" "F.Paste" "F.Mask") (roundrect_rratio 0.217391)
       (net 42 "/PoE/VSS") (pintype "passive"))
@@
     )
   )
+  (footprint "Connector_PinHeader_2.54mm:PinHeader_1x02_P2.54mm_Vertical" (layer "F.Cu")
+    (at 221.4118 92.3798)
+    (descr "Through hole straight pin header, 1x02, 2.54mm pitch, single row")
+    (tags "Through hole pin header THT 1x02 2.54mm single row")
+    (property "Description" "")
+    (property "JLCPCB Part #" "")
+    (property "Manufacturer" "")
+    (property "Partnumber" "")
+    (property "Sheetfile" "stm32f4_uno_poe.kicad_sch")
+    (property "Sheetname" "")
+    (property "exclude_from_bom" "")
+    (property "isBasicPart" "")
+    (property "ki_description" "Generic connector, single row, 01x02, script generated (kicad-library-utils/schlib/autogen/connector/)")
+    (property "ki_keywords" "connector")
+    (attr through_hole exclude_from_bom)
+    (fp_text reference "J113" (at 0 -2.33) (layer "F.SilkS")
+        (effects (font (size 1 1) (thickness 0.15)))
+    )
+    (fp_text value "Conn_01x02" (at 0 4.87) (layer "F.Fab")
+        (effects (font (size 1 1) (thickness 0.15)))
+    )
+    (fp_text user "${REFERENCE}" (at 0 1.27 90) (layer "F.Fab")
+        (effects (font (size 1 1) (thickness 0.15)))
+    )
+    (fp_line (start -1.33 -1.33) (end 0 -1.33)
+      (stroke (width 0.12) (type solid)) (layer "F.SilkS"))
+    (fp_line (start -1.33 0) (end -1.33 -1.33)
+      (stroke (width 0.12) (type solid)) (layer "F.SilkS"))
+    (fp_line (start -1.33 1.27) (end -1.33 3.87)
+      (stroke (width 0.12) (type solid)) (layer "F.SilkS"))
+    (fp_line (start -1.33 1.27) (end 1.33 1.27)
+      (stroke (width 0.12) (type solid)) (layer "F.SilkS"))
+    (fp_line (start -1.33 3.87) (end 1.33 3.87)
+      (stroke (width 0.12) (type solid)) (layer "F.SilkS"))
+    (fp_line (start 1.33 1.27) (end 1.33 3.87)
+      (stroke (width 0.12) (type solid)) (layer "F.SilkS"))
+    (fp_line (start -1.8 -1.8) (end -1.8 4.35)
+      (stroke (width 0.05) (type solid)) (layer "F.CrtYd"))
+    (fp_line (start -1.8 4.35) (end 1.8 4.35)
+      (stroke (width 0.05) (type solid)) (layer "F.CrtYd"))
+    (fp_line (start 1.8 -1.8) (end -1.8 -1.8)
+      (stroke (width 0.05) (type solid)) (layer "F.CrtYd"))
+    (fp_line (start 1.8 4.35) (end 1.8 -1.8)
+      (stroke (width 0.05) (type solid)) (layer "F.CrtYd"))
+    (fp_line (start -1.27 -0.635) (end -0.635 -1.27)
+      (stroke (width 0.1) (type solid)) (layer "F.Fab"))
+    (fp_line (start -1.27 3.81) (end -1.27 -0.635)
+      (stroke (width 0.1) (type solid)) (layer "F.Fab"))
+    (fp_line (start -0.635 -1.27) (end 1.27 -1.27)
+      (stroke (width 0.1) (type solid)) (layer "F.Fab"))
+    (fp_line (start 1.27 -1.27) (end 1.27 3.81)
+      (stroke (width 0.1) (type solid)) (layer "F.Fab"))
+    (fp_line (start 1.27 3.81) (end -1.27 3.81)
+      (stroke (width 0.1) (type solid)) (layer "F.Fab"))
+    (pad "1" thru_hole rect (at 0 0) (size 1.7 1.7) (drill 1) (layers "*.Cu" "*.Mask")
+      (net 43 "/PoE/24V") (pinfunction "Pin_1") (pintype "passive"))
+    (pad "2" thru_hole oval (at 0 2.54) (size 1.7 1.7) (drill 1) (layers "*.Cu" "*.Mask")
+      (net 1 "GND") (pinfunction "Pin_2") (pintype "passive"))
+    (model "${KICAD6_3DMODEL_DIR}/Connector_PinHeader_2.54mm.3dshapes/PinHeader_1x02_P2.54mm_Vertical.wrl"
+      (offset (xyz 0 0 0))
+      (scale (xyz 1 1 1))
+      (rotate (xyz 0 0 0))
+    )
+  )
   (footprint "Resistor_SMD:R_0603_1608Metric" (layer "F.Cu")
     (at 178.0725 64.2314)
@@
       (net 38 "/PoE/VDD") (pintype "passive"))
     (pad "2" smd roundrect (at 1.475 0) (size 1.15 1.8) (layers "F.Cu" "F.Paste" "F.Mask") (roundrect_rratio 0.217391)
-      (net 39 "/PoE/SHIELD") (pintype "passive"))
+      (net 39 "Earth") (pintype "passive"))
     (model "${KICAD6_3DMODEL_DIR}/Capacitor_SMD.3dshapes/C_1206_3216Metric.wrl"
       (offset (xyz 0 0 0))
@@
     )
   )
-  (footprint "Project_Library:Coilcraft POE40Q-xxE" (layer "F.Cu")
+  (footprint "#Transformer:Coilcraft POE40Q-xxE" (layer "F.Cu")
     (at 160.1978 79.6798 90)
     (property "Manufacturer" "Coilcraft")
@@
     (property "ki_keywords" "PCB Flyback Transformer")
     (attr smd)
-    (fp_text reference "TR201" (at 0 -8.255 90) (layer "F.SilkS") hide
+    (fp_text reference "TR201" (at 0 -8.255 90) (layer "F.SilkS")
         (effects (font (size 1 1) (thickness 0.15)))
     )
-    (fp_text value "Coilcraft POE40Q-xxE" (at 0.254 6.595 90) (layer "F.Fab") hide
+    (fp_text value "Coilcraft POE40Q-xxE" (at 0.254 6.595 90) (layer "F.Fab")
         (effects (font (size 1 1) (thickness 0.15)))
     )
@@
     (pad "10" smd rect (at 8.255 -4.962) (size 1.27 1.55) (layers "F.Cu" "F.Paste" "F.Mask")
       (net 1 "GND") (pintype "passive") (thermal_bridge_angle 45))
-    (model "${KIPRJMOD}/Project_Library.3dshapes/Coilcraft-POE40Q-XXX.step"
+    (model "${KIPRJMOD}/KiCad-Lib/#Transformer.3dshapes/Coilcraft-POE40Q-XXX.step"
       (offset (xyz 0 0 0))
       (scale (xyz 1 1 1))

Commit message: #1 Use new central library KiCad-Lib
Parts:
- J112: footprint Connector_BarrelJack:BarrelJack_CUI_PJ-102AH_Horizontal -> #Connector:CUI Devices PJ-102AH.pdf
Changed lines of the file:
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@@
     )
   )
-  (footprint "Connector_BarrelJack:BarrelJack_CUI_PJ-102AH_Horizontal" locked (layer "F.Cu")
+  (footprint "#Connector:CUI Devices PJ-102AH.pdf" locked (layer "F.Cu")
     (at 110.7948 92.3798 -90)
     (descr "Thin-pin DC Barrel Jack, https://cdn-shop.adafruit.com/datasheets/21mmdcjackDatasheet.pdf")
@@
     (property "ki_keywords" "DC power barrel jack connector")
     (attr through_hole exclude_from_bom)
-    (fp_text reference "J112" (at 5.75 8.45) (layer "F.SilkS") hide
+    (fp_text reference "J112" (at 5.75 8.45) (layer "F.SilkS")
         (effects (font (size 1 1) (thickness 0.15)))
     )
-    (fp_text value "Barrel_Jack" (at -5.5 6.2) (layer "F.Fab") hide
+    (fp_text value "Barrel_Jack" (at -5.5 6.2) (layer "F.Fab")
         (effects (font (size 1 1) (thickness 0.15)))
     )
-    (fp_text user "${REFERENCE}" (at 0 6.5 90) (layer "F.Fab") hide
+    (fp_text user "${REFERENCE}" (at 0 6.5 -90) (layer "F.Fab")
         (effects (font (size 1 1) (thickness 0.15)))
     )
@@
     (pad "3" thru_hole circle locked (at 4.7 3 270) (size 2.6 2.6) (drill 1.6) (layers "*.Cu" "*.Mask")
       (net 68 "unconnected-(J112-Pad3)") (pintype "passive+no_connect"))
-    (model "${KICAD6_3DMODEL_DIR}/Connector_BarrelJack.3dshapes/BarrelJack_CUI_PJ-102AH_Horizontal.wrl"
-      (offset (xyz 0 0 0))
+    (model "${KIPRJMOD}/KiCad-Lib/#Connector.3dshapes/CUI Devices PJ-102AH.step"
+      (offset (xyz 0 -6.5 0))
       (scale (xyz 1 1 1))
-      (rotate (xyz 0 0 0))
+      (rotate (xyz -90 0 90))
     )
   )

Commit message: WIP
Parts:
- L201, L202, L203, L204: value 600Ω@100MHz -> 100Ω@100MHz (800mA)
Changed lines of the file:
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@@
     (descr "Inductor SMD 0805 (2012 Metric), square (rectangular) end terminal, IPC_7351 nominal, (Body size source: IPC-SM-782 page 80, https://www.pcb-3d.com/wordpress/wp-content/uploads/ipc-sm-782a_amendment_1_and_2.pdf), generated with kicad-footprint-generator")
     (tags "inductor")
-    (property "Description" "300mΩ ±25% 600Ω@100MHz 0805  Ferrite Beads ROHS")
-    (property "JLCPCB Part #" "C1017")
+    (property "Description" "±25% 100Ω@100MHz 0805  Ferrite Beads ROHS")
+    (property "JLCPCB Part #" "C1015")
     (property "Manufacturer" "Sunlord")
-    (property "Manufacturer_Name" "Sunlord")
-    (property "Manufacturer_Part_Number" "GZ2012D601TF")
-    (property "Partnumber" "GZ2012D601TF")
+    (property "Partnumber" "GZ2012D101TF")
     (property "Sheetfile" "poe.kicad_sch")
     (property "Sheetname" "PoE")
@@
         (effects (font (size 0.8 0.8) (thickness 0.15)))
     )
-    (fp_text value "600Ω@100MHz" (at 0 1.55) (layer "F.Fab") hide
+    (fp_text value "100Ω@100MHz (800mA)" (at 0 1.55) (layer "F.Fab") hide
         (effects (font (size 0.8 0.8) (thickness 0.15)))
     )
@@
         (effects (font (size 1 1) (thickness 0.15)))
     )
-    (fp_text user "${REFERENCE}" (at 0 6.5 -90) (layer "F.Fab")
+    (fp_text user "${REFERENCE}" (at 0 6.5 90) (layer "F.Fab")
         (effects (font (size 1 1) (thickness 0.15)))
     )
@@
     (descr "Inductor SMD 0805 (2012 Metric), square (rectangular) end terminal, IPC_7351 nominal, (Body size source: IPC-SM-782 page 80, https://www.pcb-3d.com/wordpress/wp-content/uploads/ipc-sm-782a_amendment_1_and_2.pdf), generated with kicad-footprint-generator")
     (tags "inductor")
-    (property "Description" "300mΩ ±25% 600Ω@100MHz 0805  Ferrite Beads ROHS")
-    (property "JLCPCB Part #" "C1017")
+    (property "Description" "±25% 100Ω@100MHz 0805  Ferrite Beads ROHS")
+    (property "JLCPCB Part #" "C1015")
     (property "Manufacturer" "Sunlord")
-    (property "Manufacturer_Name" "Sunlord")
-    (property "Manufacturer_Part_Number" "GZ2012D601TF")
-    (property "Partnumber" "GZ2012D601TF")
+    (property "Partnumber" "GZ2012D101TF")
     (property "Sheetfile" "poe.kicad_sch")
     (property "Sheetname" "PoE")
@@
         (effects (font (size 0.8 0.8) (thickness 0.15)))
     )
-    (fp_text value "600Ω@100MHz" (at 0 1.55) (layer "F.Fab") hide
+    (fp_text value "100Ω@100MHz (800mA)" (at 0 1.55) (layer "F.Fab") hide
         (effects (font (size 0.8 0.8) (thickness 0.15)))
     )
@@
     (descr "Inductor SMD 0805 (2012 Metric), square (rectangular) end terminal, IPC_7351 nominal, (Body size source: IPC-SM-782 page 80, https://www.pcb-3d.com/wordpress/wp-content/uploads/ipc-sm-782a_amendment_1_and_2.pdf), generated with kicad-footprint-generator")
     (tags "inductor")
-    (property "Description" "300mΩ ±25% 600Ω@100MHz 0805  Ferrite Beads ROHS")
-    (property "JLCPCB Part #" "C1017")
+    (property "Description" "±25% 100Ω@100MHz 0805  Ferrite Beads ROHS")
+    (property "JLCPCB Part #" "C1015")
     (property "Manufacturer" "Sunlord")
-    (property "Manufacturer_Name" "Sunlord")
-    (property "Manufacturer_Part_Number" "GZ2012D601TF")
-    (property "Partnumber" "GZ2012D601TF")
+    (property "Partnumber" "GZ2012D101TF")
     (property "Sheetfile" "poe.kicad_sch")
     (property "Sheetname" "PoE")
@@
         (effects (font (size 0.8 0.8) (thickness 0.15)))
     )
-    (fp_text value "600Ω@100MHz" (at 0 1.55) (layer "F.Fab") hide
+    (fp_text value "100Ω@100MHz (800mA)" (at 0 1.55) (layer "F.Fab") hide
         (effects (font (size 0.8 0.8) (thickness 0.15)))
     )
@@
     (descr "Inductor SMD 0805 (2012 Metric), square (rectangular) end terminal, IPC_7351 nominal, (Body size source: IPC-SM-782 page 80, https://www.pcb-3d.com/wordpress/wp-content/uploads/ipc-sm-782a_amendment_1_and_2.pdf), generated with kicad-footprint-generator")
     (tags "inductor")
-    (property "Description" "300mΩ ±25% 600Ω@100MHz 0805  Ferrite Beads ROHS")
-    (property "JLCPCB Part #" "C1017")
+    (property "Description" "±25% 100Ω@100MHz 0805  Ferrite Beads ROHS")
+    (property "JLCPCB Part #" "C1015")
     (property "Manufacturer" "Sunlord")
-    (property "Manufacturer_Name" "Sunlord")
-    (property "Manufacturer_Part_Number" "GZ2012D601TF")
-    (property "Partnumber" "GZ2012D601TF")
+    (property "Partnumber" "GZ2012D101TF")
     (property "Sheetfile" "poe.kicad_sch")
     (property "Sheetname" "PoE")
@@
         (effects (font (size 0.8 0.8) (thickness 0.15)))
     )
-    (fp_text value "600Ω@100MHz" (at 0 1.55) (layer "F.Fab") hide
+    (fp_text value "100Ω@100MHz (800mA)" (at 0 1.55) (layer "F.Fab") hide
         (effects (font (size 0.8 0.8) (thickness 0.15)))
     )
