File: poe.kicad_sch (KiCad schematic)
At the start: 45 parts

Commit message: WIP
Parts:
- added C1: 22u 25V, Capacitor_SMD:C_0805_2012Metric, symbol Device:C_Small
- added C1 (x3): 2u2 100V, Capacitor_SMD:C_1206_3216Metric, symbol Device:C_Small
- added C125: 100n 100V, Capacitor_SMD:C_0805_2012Metric, symbol Device:C_Small
- added C125: 100p 500V, Capacitor_SMD:C_0805_2012Metric, symbol Device:C_Small
- added C211: 47u 63V, Capacitor_SMD:C_Elec_8x10.2, symbol Device:C_Polarized_Small
- added D205: 1A 200V 35ns, Diode_SMD:D_SMA, symbol Device:D_Small
- added D8: 1N4148WS, Diode_SMD:D_SOD-323, symbol Device:D_Small
- added L205: 3u3, Inductor_SMD:L_Sunlord_SWPA4030S, symbol Device:L_Small
- added Q201: Si7450DP, Package_SO:PowerPAK_SO-8_Single, symbol Transistor_FET:Si7450DP
- added R123: 4E7, Resistor_SMD:R_0603_1608Metric, symbol Device:R_Small
- added R123: 39k, Resistor_SMD:R_0805_2012Metric, symbol Device:R_Small
- added R123: 100, Resistor_SMD:R_0603_1608Metric, symbol Device:R_Small
- added R123: 274k, Resistor_SMD:R_0603_1608Metric, symbol Device:R_Small
- added R123: 0E12 1W, Resistor_SMD:R_2512_6332Metric, symbol Device:R_Small
- added R123: 1k, Resistor_SMD:R_0603_1608Metric, symbol Device:R_Small
- added R123: 75 750mW, Resistor_SMD:R_2010_5025Metric, symbol Device:R_Small
Connections:
- net PGND: now also C1.2, C1.2, C1.2, C1.2, C211.2, R123.2, R123.2
- net VDD: now also C1.1, C211.1, L205.1, R123.1
- net CS: now reaches U?.3 (CS)
- net CS: now also R123.2, R123.2
- net GATE: now reaches U?.5 (GATE)
- net GATE: now also R123.2, R123.2
- net VC: now reaches C?.1, U?.6 (VC)
- net VC: now also C1.1
- new net: D8.1 (K), R123.1
- new net: C1.1, C1.1, C125.1, L205.2, R123.1
- new net: C125.2, D205.1 (K), R123.2
- new net: D8.2 (A), Q201.4 (G), R123.1
- new net: Q201.1 (S), Q201.2 (S), Q201.3 (S), R123.1, R123.1
- new net: C125.1, D205.2 (A), Q201.5 (D)
- new net: C125.2, R123.1
Other:
- note removed: "PoE"

Commit message: Add flyback transformator
Parts:
- added TR201: Coilcraft POE40Q-xxE, Project_Library:Coilcraft POE40Q-xxE, symbol Project_Library:Coilcraft POE40Q-xxE
Changed lines of the file:
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@@
+    )
+  )
+  (symbol (lib_id "Project_Library:Coilcraft POE40Q-xxE") (at 121.92 118.745 0) (unit 1)
+    (in_bom yes) (on_board yes) (dnp no) (fields_autoplaced)
+    (property "Reference" "TR201" (at 123.2505 105.41 0)
+      (effects (font (size 1.27 1.27)))
+    )
+    (property "Value" "Coilcraft POE40Q-xxE" (at 123.2505 107.95 0)
+      (effects (font (size 1.27 1.27)))
+    )
+    (property "Footprint" "Project_Library:Coilcraft POE40Q-xxE" (at 121.92 132.715 0)
+      (effects (font (size 1.27 1.27)) hide)
+    )
+    (property "Datasheet" "https://www.coilcraft.com/getmedia/71a3c6d3-d040-4587-8bbd-dd1492f81afc/poexxq.pdf" (at 121.92 118.745 0)
+      (effects (font (size 1.27 1.27)) hide)
+    )
+    (property "Manufacturer" "Coilcraft" (at 121.92 137.795 0)
+      (effects (font (size 1.27 1.27)) hide)
+    )
+    (pin "1")
+    (pin "10")
+    (pin "2")
+    (pin "3")
+    (pin "4")
+    (pin "5")
+    (pin "6")
+    (pin "7")
+    (pin "8")
+    (pin "9")
+    (instances
+      (project "stm32f4_uno_poe"
+        (path "/e63e39d7-6ac0-4ffd-8aa3-1841a4541b55/6d67357d-4810-4134-a5e5-d0bcd5308ea5"
+          (reference "TR201") (unit 1)
+        )
+      )
     )
   )

Commit message: WIP
Parts:
- added C133 (x2): 1u 50V, Capacitor_SMD:C_0603_1608Metric, symbol Device:C_Small
- added C133 (x4): 1n 2kV, Capacitor_SMD:C_1206_3216Metric, symbol Device:C_Small
- added C133 (x4): 4u7 50V, Capacitor_SMD:C_1206_3216Metric, symbol Device:C_Small
- added C231: 22u 63V, Capacitor_SMD:C_Elec_6.3x5.4, symbol Device:C_Polarized_Small
- added C?: 330p 500V, Capacitor_SMD:C_0805_2012Metric, symbol Device:C_Small
- added D208: 150V 10A, Package_TO_SOT_SMD:TO-277A, symbol Device:D_Schottky_AAK
- added D8: 1N4148WS, Diode_SMD:D_SOD-323, symbol Device:D_Small
- added R123 (x2): 100 750mW, Resistor_SMD:R_2010_5025Metric, symbol Device:R_Small
- added R123: 20, Resistor_SMD:R_0805_2012Metric, symbol Device:R_Small
- added R?: 10k, Resistor_SMD:R_0603_1608Metric, symbol Device:R_Small
- added U204: EL357N(C)(TA)-G, Package_SO:SOP-4_3.8x4.1mm_P2.54mm, symbol Isolator:FODM217D
- R123: Manufacturer FOJAN -> Walsin Tech Corp
Connections:
- net 24V: now also C133.1, C133.1, C133.1, C133.1, C133.1, C231.1, C?.1, D208.3 (K)
- net GND: now also TR201.10, TR201.9, C133.2, C133.2, C133.2, C133.2, C133.2, C133.2, C133.2, C133.2, C133.2, C231.2
- net PGND: now also TR201.4, C133.1, C133.1, C133.2
- net T2P: now also U204.2
- net VC: now also C133.1, D8.1 (K), R?.2
- net at C1.1, C1.1, C125.1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: now also TR201.1, C133.1, C133.1
- net at TR201.3: now also C125.1, D205.2 (A), Q201.5 (D)
- net at TR201.5: now also R123.1
- net at TR201.6: now also TR201.7, D208.1 (A), D208.2 (A), R123.1, R123.1
- new net: R?.1, U204.1
- new net: C?.2, R123.2, R123.2
- new net: D8.2 (A), R123.2
- no-connect marks 1 -> 4
Other:
- moved on the sheet: C125, D205, D8, Q201, R123, TR201

Commit message: #1 Use new central library KiCad-Lib
Parts:
- TR201: footprint Project_Library:Coilcraft POE40Q-xxE -> #Transformer:Coilcraft POE40Q-xxE; symbol Project_Library:Coilcraft POE40Q-xxE -> #Transformer:Coilcraft POE40Q-xxE
- U?: symbol Project_Library:TI TPS23754PWP -> #IC:Texas Instruments TPS23754PWP
Changed lines of the file:
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@@
     )
   )
-  (symbol (lib_id "Project_Library:TI TPS23754PWP") (at 128.27 57.15 0) (unit 1)
+  (symbol (lib_id "#IC:Texas Instruments TPS23754PWP") (at 128.27 57.15 0) (unit 1)
     (in_bom yes) (on_board yes) (dnp no) (fields_autoplaced)
-    (property "Reference" "U?" (at 143.51 50.165 0)
-      (effects (font (size 1 1)))
-    )
-    (property "Value" "TPS23754PWP" (at 143.51 52.705 0)
+    (property "Reference" "U?" (at 143.51 49.53 0)
+      (effects (font (size 1 1)))
+    )
+    (property "Value" "TPS23754PWP" (at 143.51 52.07 0)
       (effects (font (size 1 1)))
     )
     (property "Footprint" "Package_SO:TSSOP-20-1EP_4.4x6.5mm_P0.65mm_EP2.15x3.35mm" (at 154.94 152.07 0)
-      (effects (font (size 1 1)) (justify left top) hide)
-    )
-    (property "Datasheet" "http://www.ti.com/lit/gpn/tps23754" (at 154.94 252.07 0)
-      (effects (font (size 1 1)) (justify left top) hide)
+      (effects (font (size 1.27 1.27)) (justify left top) hide)
+    )
+    (property "Datasheet" "${KIPRJMOD}/KiCad-Lib/#IC.doc/Texas Instruments TPS23754PWP.pdf" (at 154.94 252.07 0)
+      (effects (font (size 1.27 1.27)) (justify left top) hide)
     )
     (property "Manufacturer" "Texas Instruments" (at 154.94 752.07 0)
-      (effects (font (size 1 1)) (justify left top) hide)
+      (effects (font (size 1.27 1.27)) (justify left top) hide)
     )
     (property "Partnumber" "TPS23754PWP" (at 154.94 852.07 0)
-      (effects (font (size 1 1)) (justify left top) hide)
+      (effects (font (size 1.27 1.27)) (justify left top) hide)
     )
     (property "JLCPCB Part #" "C181651" (at 143.51 106.934 0) (show_name)
-      (effects (font (size 1 1)) hide)
+      (effects (font (size 1.27 1.27)) hide)
     )
     (property "isBasicPart" "NO" (at 143.51 109.22 0) (show_name)
-      (effects (font (size 1 1)) hide)
+      (effects (font (size 1.27 1.27)) hide)
     )
     (property "Description" "TSSOP-20-EP  Power Over Ethernet Controllers ROHS" (at 143.764 104.902 0)
-      (effects (font (size 1 1)) hide)
+      (effects (font (size 1.27 1.27)) hide)
     )
     (pin "1")
@@
     )
   )
-  (symbol (lib_id "Project_Library:Coilcraft POE40Q-xxE") (at 137.795 115.57 0) (unit 1)
+  (symbol (lib_id "#Transformer:Coilcraft POE40Q-xxE") (at 137.795 115.57 0) (unit 1)
     (in_bom yes) (on_board yes) (dnp no) (fields_autoplaced)
-    (property "Reference" "TR201" (at 139.1255 102.235 0)
+    (property "Reference" "TR201" (at 139.1255 102.87 0)
       (effects (font (size 1.27 1.27)))
     )
-    (property "Value" "Coilcraft POE40Q-xxE" (at 139.1255 104.775 0)
+    (property "Value" "Coilcraft POE40Q-xxE" (at 139.1255 105.41 0)
       (effects (font (size 1.27 1.27)))
     )
-    (property "Footprint" "Project_Library:Coilcraft POE40Q-xxE" (at 137.795 129.54 0)
+    (property "Footprint" "#Transformer:Coilcraft POE40Q-xxE" (at 137.795 129.54 0)
       (effects (font (size 1.27 1.27)) hide)
     )
-    (property "Datasheet" "https://www.coilcraft.com/getmedia/71a3c6d3-d040-4587-8bbd-dd1492f81afc/poexxq.pdf" (at 137.795 115.57 0)
+    (property "Datasheet" "${KIPRJMOD}/KiCad-Lib/#Transformer.doc/poexxq.pdf" (at 137.795 136.906 0)
       (effects (font (size 1.27 1.27)) hide)
     )

Commit message: WIP
Parts:
- removed L? (x4): 600Ω@100MHz, Inductor_SMD:L_0805_2012Metric, symbol Device:FerriteBead_Small
- added L101 (x4): 100Ω@100MHz (800mA), Inductor_SMD:L_0805_2012Metric, symbol Device:FerriteBead_Small
Connections:
- net AUX: now also L101.2
- net PGND: now also L101.2
- net VDD: now also L101.2
- net VDD_B: now also L101.1
- net VSS: now also L101.2
- net VSS_B: now also L101.1
- net V_{AUX}+: now also L101.1
- net V_{AUX}-: now also L101.1
Other:
- moved on the sheet: C?, D?

Commit message: WIP
Parts:
- removed R?: 4k7, Resistor_SMD:R_0402_1005Metric, symbol Device:R_Small
- removed R?: 200, Resistor_SMD:R_0402_1005Metric, symbol Device:R_Small
- removed R?: 20k, Resistor_SMD:R_0402_1005Metric, symbol Device:R_Small
- added R123: 10k, Resistor_SMD:R_0603_1608Metric, symbol Device:R_Small
- added R123: 15k, Resistor_SMD:R_0603_1608Metric, symbol Device:R_Small
Connections:
- net VDD: now also R123.1
- net at U?.13 (DEN): now also R123.2
- new net: R123.1, R123.2

Commit message: WIP
Parts:
- D205: value 1A 200V 35ns -> 1A 1kV 75ns; JLCPCB Part # C116492 -> C412437; Manufacturer Shandong Jingdao Microelectronics -> MDD; Partnumber ES1D -> US1M; isBasicPart NO -> YES
- D8: isBasicPart NO -> YES
- D?: value SS210 -> SS220; JLCPCB Part # C14996 -> C7420361; Manufacturer_Name MDD -> (none); Manufacturer_Part_Number SS210 -> (none)
- D?: JLCPCB Part # (none) -> C7420333; Manufacturer (none) -> hongjiacheng; Partnumber (none) -> BAT54S; isBasicPart (none) -> YES
- U?: value TCMT1107 -> EL3H7(A)(TA)-G; JLCPCB Part # (none) -> C181879; Manufacturer (none) -> Everlight Elec; Partnumber (none) -> EL3H7(A)(TA)-G; isBasicPart (none) -> NO
Connections:
- net CTL: now also U?.4; no longer U?.1
- net PGND: now also U?.3; no longer U?.2
- net at C?.2, D?.1 (A), R?.1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: now also U?.2; no longer U?.3
- net at R?.2: now also U?.1; no longer U?.4
Other:
- moved on the sheet: C1, C133, C211, C?, D8, D?, R123, R?, U204, U?

Commit message: WIP
Parts:
- removed C? (x2): 1n 2kV, Capacitor_SMD:C_1206_3216Metric, symbol Device:C_Small
- removed L101 (x4): 100Ω@100MHz (800mA), Inductor_SMD:L_0805_2012Metric, symbol Device:FerriteBead_Small
- removed R?: 68, Resistor_SMD:R_0805_2012Metric, symbol Device:R_Small
- removed R?: 1k, Resistor_SMD:R_0805_2012Metric, symbol Device:R_Small
- added D?: 58V TVS, Diode_SMD:D_SMB, symbol Device:D_Schottky_Small
- added L101 (x4): 600Ω@100MHz (500mA), Inductor_SMD:L_0805_2012Metric, symbol Device:FerriteBead_Small
- added R2 (x2): 470, Resistor_SMD:R_0402_1005Metric, symbol Device:R_Small
- added R2: 330, Resistor_SMD:R_0402_1005Metric, symbol Device:R_Small
- added TP201: VDD, TestPoint:TestPoint_THTPad_2.0x2.0mm_Drill1.0mm, symbol Connector:TestPoint
- added TP202: VSS, TestPoint:TestPoint_THTPad_2.0x2.0mm_Drill1.0mm, symbol Connector:TestPoint
- D?: value 64V TVS -> 58V TVS; footprint Diode_SMD:D_SMC -> Diode_SMD:D_SMA; JLCPCB Part # C2990414 -> C115922; Manufacturer Liown -> Brightking; Manufacturer_Name Liown -> (none); Manufacturer_Part_Number 5.0SMDJ64CA -> (none); Partnumber 5.0SMDJ64CA -> SMAJ58A/TR13; isBasicPart YES -> NO
- D? (x2): Manufacturer_Name MDD -> (none); Manufacturer_Part_Number MB10S -> (none)
Connections:
- net 24V: no longer C133.1, C133.1, C133.1, C133.1, C133.1, C231.1, C?.1, D208.3 (K)
- net AUX: now also L101.2
- net PGND: now also D?.1 (K), L101.2
- net VDD: now also L101.2, TP201.1
- net VDD_B: now also L101.1
- net VSS: now also D?.2 (A), L101.2, R2.1, TP202.1
- net VSS_B: now also L101.1
- net V_{AUX}+: now also L101.1
- net V_{AUX}-: now also L101.1
- net +V_SEC: now reaches D208.1 (A), D208.2 (A), R123.1, R123.1, TR201.6, TR201.7
- net at U?.15 (CLS): now also R2.2
- net VDD_PRI+: now reaches C1.1, C1.1, C125.1, C133.1, C133.1, L205.2, R123.1, TR201.1
- net VDD_SN: now reaches C125.2, D205.1 (K), R123.2
- net VDD_PRI-: now reaches C125.1, D205.2 (A), Q201.5 (D), TR201.3
- net PGND_S: now reaches Q201.1 (S), Q201.2 (S), Q201.3 (S), R123.1, R123.1
- new net: R2.1, R2.2 (x2)
- new net +24V: C133.1, C133.1, C133.1, C133.1, C133.1, C231.1, C?.1, D208.3 (K)
- no-connect marks 4 -> 5
