File: poe.kicad_sch (KiCad schematic)
At the start: 84 parts, among them Q201 Si7450DP, U204 EL357N(C)(TA)-G

Commit message: PCB ready
Parts:
- removed R?: 10k, Resistor_SMD:R_0603_1608Metric, symbol Device:R_Small
- removed U204: EL357N(C)(TA)-G, Package_SO:SOP-4_3.8x4.1mm_P2.54mm, symbol Isolator:FODM217D
- added D1: LED green, LED_SMD:LED_0603_1608Metric, symbol Device:LED_Small
- added R123: 4k7, Resistor_SMD:R_0402_1005Metric, symbol Device:R_Small
- TR201: value Coilcraft POE40Q-xxE -> Coilcraft POE40Q-24E; now left out of the parts list
Connections:
- net 24V is gone; now on net +24V: D?.2 (K), R?.1, R?.1, R?.1, R?.1
- net T2P: now also D1.1 (K)
- net VC: now also R123.2
- new net: D1.2 (A), R123.1
- no-connect marks 5 -> 3

Commit message: #2 Add silkscreen texts
Other:
- company: (none) -> easy-smart solution GmbH
- title: (none) -> STM32F4 Uno PoE
Changed lines of the file:
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@@
   (paper "A4")
   (title_block
-    (date "2023-09-07")
+    (title "STM32F4 Uno PoE")
+    (date "2023-10-02")
+    (rev "1.0.x-dev")
+    (company "easy-smart solution GmbH")
   )
   (junction (at 37.465 29.21) (diameter 0) (color 0 0 0 0)

Commit message: Release 1.0.0 sent to JLCPCB
Parts:
- D?: Partnumber SS210 -> SS220
Changed lines of the file:
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@@
     (title "STM32F4 Uno PoE")
     (date "2023-10-02")
-    (rev "1.0.x-dev")
+    (rev "1.0.0")
     (company "easy-smart solution GmbH")
   )
@@
       (effects (font (size 1 1)) hide)
     )
-    (property "Partnumber" "SS210" (at 65.405 29.21 0)
-      (effects (font (size 1 1)) hide)
-    )
+    (property "Partnumber" "SS220" (at 65.405 29.21 0)
+      (effects (font (size 1 1)) hide)
+    )
