File: stm32f4_uno_poe.kicad_sch (KiCad schematic)
At the start: 13 parts, among them J101 STM32 GPIO, J102 Digital/PWM, J103 STM32 GPIO, J104 STM32 GPIO, J105 STM32 GPIO, J106 Power, J107 Conn_01x04, J108 Ethernet, J109 STM32 GPIO, J110 Digital/PWM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

Commit message: WIP
Other:
- note removed: "* Indicates a PWM-capable pin"
Changed lines of the file:
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@@
     (effects (font (size 1 1)) (justify right bottom))
-  )
-  (text "* Indicates a PWM-capable pin" (at 177.8 180.34 0)
-    (effects (font (size 1.27 1.27)) (justify left bottom))
   )
   (text "TX/D1" (at 280.035 75.565 0)

Commit message: PCB ready
Parts:
- J104, J108, J111: now not fitted
Connections:
- net GND: no longer J104.1 (Pin_1)
Changed lines of the file:
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@@
   )
   (symbol (lib_id "Connector_Generic:Conn_01x06") (at 189.865 70.485 0) (unit 1)
-    (in_bom no) (on_board yes) (dnp no)
+    (in_bom no) (on_board no) (dnp yes)
     (property "Reference" "J111" (at 189.865 62.865 0)
       (effects (font (size 0.9 0.9)))
@@
   )
   (symbol (lib_id "Connector_Generic:Conn_01x10") (at 242.57 65.405 0) (mirror y) (unit 1)
-    (in_bom no) (on_board yes) (dnp no)
+    (in_bom no) (on_board no) (dnp yes)
     (property "Reference" "J108" (at 242.57 52.705 0)
       (effects (font (size 0.9 0.9)))
@@
   )
   (symbol (lib_id "Connector_Generic:Conn_01x08") (at 242.57 39.37 0) (mirror y) (unit 1)
-    (in_bom no) (on_board yes) (dnp no)
+    (in_bom no) (on_board no) (dnp yes)
     (property "Reference" "J104" (at 242.57 29.21 0)
       (effects (font (size 0.9 0.9)))
@@
         )
       )
-    )
-  )
-  (symbol (lib_id "power:GND") (at 247.65 31.75 90) (unit 1)
-    (in_bom yes) (on_board yes) (dnp no)
-    (property "Reference" "#PWR0106" (at 254 31.75 0)
-      (effects (font (size 0.9 0.9)) hide)
-    )
-    (property "Value" "GND" (at 252.095 31.75 90)
-      (effects (font (size 0.9 0.9)))
-    )
-    (property "Footprint" "" (at 247.65 31.75 0)
-      (effects (font (size 1 1)))
-    )
-    (property "Datasheet" "" (at 247.65 31.75 0)
-      (effects (font (size 1 1)))
-    )
-    (pin "1")
-    (instances
-      (project "stm32f4_uno_poe"
-        (path "/e63e39d7-6ac0-4ffd-8aa3-1841a4541b55"
-          (reference "#PWR0106") (unit 1)
-        )
-      )

Commit message: #2 Add silkscreen texts
Parts:
- added D8: SS210, Diode_SMD:D_SMA, symbol Device:D_Schottky_Small
Connections:
- net PoE/+24V: now also D8.2 (A); no longer J106.8 (Pin_8)
- new net: D8.1 (K), J106.8 (Pin_8)
Other:
- company: (none) -> easy-smart solution GmbH
- title: (none) -> STM32F4 Uno PoE
Changed lines of the file:
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@@
   (paper "A4")
   (title_block
-    (date "mar. 31 mars 2015")
+    (title "STM32F4 Uno PoE")
+    (date "2023-10-02")
+    (rev "1.0.x-dev")
+    (company "easy-smart solution GmbH")
   )
   (junction (at 176.53 45.085) (diameter 0) (color 0 0 0 0)
@@
     (stroke (width 0) (type default))
   )
-  (wire (pts (xy 121.92 55.245) (xy 184.785 55.245))
+  (wire (pts (xy 121.92 55.245) (xy 144.145 55.245))
     (stroke (width 0) (type default))
   )
@@
   (wire (pts (xy 267.335 75.565) (xy 280.035 75.565))
     (stroke (width 0) (type solid))
+  )
+  (wire (pts (xy 149.225 55.245) (xy 184.785 55.245))
+    (stroke (width 0) (type default))
   )
   (wire (pts (xy 184.785 75.565) (xy 172.085 75.565))
@@
         )
       )
+    )
+  )
+  (symbol (lib_id "Device:D_Schottky_Small") (at 146.685 55.245 180) (unit 1)
+    (in_bom yes) (on_board yes) (dnp no) (fields_autoplaced)
+    (property "Reference" "D8" (at 146.939 48.895 0)
+      (effects (font (size 0.9 0.9)))
+    )
+    (property "Value" "SS210" (at 146.939 51.435 0)
+      (effects (font (size 0.9 0.9)))
+    )
+    (property "Footprint" "Diode_SMD:D_SMA" (at 146.685 55.245 90)
+      (effects (font (size 1 1)) hide)
+    )
+    (property "Datasheet" "https://datasheet.lcsc.com/lcsc/2304140030_MDD-Microdiode-Electronics--SS210_C14996.pdf" (at 146.685 55.245 90)
+      (effects (font (size 1 1)) hide)
+    )
+    (property "Description" "100V 850mV@2A 2A SMA(DO-214AC)  Schottky Barrier Diodes (SBD) ROHS" (at 146.685 55.245 0)
+      (effects (font (size 1 1)) hide)
+    )
+    (property "Manufacturer" "MDD" (at 146.685 55.245 0)
+      (effects (font (size 1 1)) hide)
+    )
+    (property "Partnumber" "SS210" (at 146.685 55.245 0)
+      (effects (font (size 1 1)) hide)
+    )
+    (property "JLCPCB Part #" "C14996" (at 146.685 55.245 0)
+      (effects (font (size 1 1)) hide)
+    )
+    (property "isBasicPart" "YES" (at 146.685 55.245 0)
+      (effects (font (size 1 1)) hide)
+    )
+    (pin "1")
+    (pin "2")
+    (instances
+      (project "stm32f1_nano"
+        (path "/0d35483a-0b12-46cc-b9f2-896fd6831779"
+          (reference "D8") (unit 1)
+        )
+      )
+      (project "stm32f407vg"
+        (path "/2d452db2-a0cd-4a57-9497-df1dd0591a30/50c2bb91-d0dc-4111-959e-b2cc7ea59413"
+          (reference "D601") (unit 1)
+        )
+      )
+      (project "basicparts"
+        (path "/43a31acf-2604-4bbd-9556-e633c3dff6c4"
+          (reference "D102") (unit 1)
+        )
+      )
+      (project "stm32f4_uno_poe"
+        (path "/e63e39d7-6ac0-4ffd-8aa3-1841a4541b55"
+          (reference "D101") (unit 1)
+        )
+      )

Commit message: Release 1.0.0 sent to JLCPCB
Parts:
- J109, J110: now fitted
Changed lines of the file:
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@@
     (title "STM32F4 Uno PoE")
     (date "2023-10-02")
-    (rev "1.0.x-dev")
+    (rev "1.0.0")
     (company "easy-smart solution GmbH")
   )
@@
   )
   (symbol (lib_id "Connector_Generic:Conn_01x08") (at 262.255 67.945 0) (mirror y) (unit 1)
-    (in_bom no) (on_board no) (dnp yes)
+    (in_bom no) (on_board yes) (dnp no)
     (property "Reference" "J110" (at 262.255 57.785 0)
       (effects (font (size 0.9 0.9)))
@@
   )
   (symbol (lib_id "Connector_Generic:Conn_01x06") (at 204.47 67.945 0) (unit 1)
-    (in_bom no) (on_board no) (dnp yes)
+    (in_bom no) (on_board yes) (dnp no)
     (property "Reference" "J109" (at 204.47 60.325 0)
       (effects (font (size 0.9 0.9)))
